File: ai03-pcb-guide.kicad_pcb (KiCad board)
At the start: 2 copper layers, 69.1 x 38.1 mm, 24 parts, among them U1 ATmega32U4-AU

Commit message: Final Touches
Ready to be printed and made.
Routing:
- added copper zone on F.Cu, net GND
Other:
- outline, holes or cut-outs redrawn
